File: circuit/mb/mb.kicad_pcb (KiCad board)
At the start: 2 copper layers, 100.6 x 69.9 mm, 50 parts, among them J1 Conn_01x03_Male, J10 Conn_01x02_Male, J2 Conn_01x02_Male, J3 Barrel_Jack_Switch, J4 Conn_02x03_Odd_Even, J5 Conn_01x04_Male, J6 Conn_01x04_Male, J7 Conn_01x04_Male, J8 Conn_01x05_Male, J9 Conn_01x05_Male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

Commit message: Add dxf and bom
Parts:
- J10: value Conn_01x02_Male -> Conn_01x03_Male; footprint Connector_PinHeader_2.54mm:PinHeader_1x02_P2.54mm_Vertical -> Connector_PinHeader_2.54mm:PinHeader_1x03_P2.54mm_Vertical
- moved R6 15.5 mm to (40.4, 69.8), turned to 0 degrees
- moved J10 3.21 mm to (42.9, 66.8)
Connections:
- R6 pad 1: NRST -> GND
- R6 pad 2: GND -> Net-(J10-Pad3)
Routing:
- net GND: track 344.8 -> 329.2 mm
- net Net-(J10-Pad3): track 0.00 -> 3.05 mm
- net +5V: track 207.0 -> 209.6 mm
- net NRST: track 26.7 -> 27.6 mm
Other:
- net class Default: trace_width 0.8 -> 0.6
- board text added: "TODO: FIX NRST BEHAVIOUR"
- board text added: "Счетометр 1.3"
- board text removed: "Счетометр 1.2"
