File: circuit/schematic.kicad_pcb (KiCad board)
At the start: 2 copper layers, 127.2 x 85.4 mm, 62 parts, among them J1 Barrel_Jack_Switch, J2 Conn_01x05_Male, J3 AudioJack3, J4 Conn_01x02_Male, SW1 SW_DPDT_x2, SW2 Rotary_Encoder_Switch, SW3 SW_Push, SW4 SW_Push, SW5 SW_Push, U1 ATmega328-AU, U2 MC33063AD, U3 SSM2211S, U4 STP08CP05, U5 74HC14, U6 CC56-12SRWA, Y1 16M

Commit message: Update board
Parts:
- removed BT1: 9V, Connector_PinHeader_2.54mm:PinHeader_1x02_P2.54mm_Vertical
- removed the C2 at (126.3, 22.5)
- removed the C8 at (139.9, 45.7)
- removed the D3 at (162.8, 23.1)
- removed LS1: Speaker, Connector_PinHeader_2.54mm:PinHeader_1x02_P2.54mm_Vertical
- removed the R22 at (125.8, 58.0)
- removed the SW1 at (109.5, 88.5)
- added C10: 220u, Capacitor_THT:CP_Radial_D8.0mm_P3.50mm, F.Cu at (263.9, 46.2)
- added C11: 220u, Capacitor_THT:CP_Radial_D8.0mm_P3.50mm, F.Cu at (276.1, 46.2)
- added C13: 0.1u, Capacitor_SMD:C_0603_1608Metric_Pad1.05x0.95mm_HandSolder, B.Cu at (258.7, 36.4)
- added C3: 220u, Capacitor_THT:CP_Radial_D8.0mm_P3.50mm, F.Cu at (270.4, 74.4)
- added C5: 100u, Capacitor_THT:CP_Radial_D8.0mm_P3.50mm, B.Cu at (276.1, 37.6)
- added C6: 0.1u, Capacitor_SMD:C_0603_1608Metric_Pad1.05x0.95mm_HandSolder, B.Cu at (266.0, 66.7)
- added D2: LED, LED_THT:LED_D3.0mm, F.Cu at (266.6, 17.2)
- added H1: MountingHole, MountingHole:MountingHole_3.2mm_M3, F.Cu at (271.7, 16.9)
- added H2: MountingHole, MountingHole:MountingHole_3.2mm_M3, F.Cu at (226.8, 76.4)
- added H3: MountingHole, MountingHole:MountingHole_3.2mm_M3, F.Cu at (279.7, 76.4)
- added H4: MountingHole, MountingHole:MountingHole_3.2mm_M3, F.Cu at (234.8, 16.9)
- added R1: 5k, Resistor_SMD:R_0603_1608Metric_Pad1.05x0.95mm_HandSolder, B.Cu at (266.0, 68.2)
- added R11: 4.7k, Resistor_SMD:R_0603_1608Metric_Pad1.05x0.95mm_HandSolder, B.Cu at (277.6, 56.0)
- added R12: 4.7k, Resistor_SMD:R_0603_1608Metric_Pad1.05x0.95mm_HandSolder, B.Cu at (277.6, 52.6)
- added R9: 5k, Resistor_SMD:R_0603_1608Metric_Pad1.05x0.95mm_HandSolder, B.Cu at (239.8, 37.5)
- added RV1: R_POT_Dual, Potentiometer_THT:Potentiometer_Alps_RK09L_Double_Vertical, F.Cu at (268.9, 54.6)
- C1: footprint Capacitor_SMD:C_0805_2012Metric_Pad1.15x1.40mm_HandSolder -> Capacitor_SMD:C_0603_1608Metric
- C14: renamed from C10; footprint Capacitor_SMD:C_0805_2012Metric_Pad1.15x1.40mm_HandSolder -> Capacitor_SMD:C_0603_1608Metric_Pad1.05x0.95mm_HandSolder
- C15: renamed from C11; footprint Capacitor_SMD:C_0805_2012Metric_Pad1.15x1.40mm_HandSolder -> Capacitor_SMD:C_0603_1608Metric_Pad1.05x0.95mm_HandSolder
- C16: renamed from C12; footprint Capacitor_SMD:C_0805_2012Metric_Pad1.15x1.40mm_HandSolder -> Capacitor_SMD:C_0603_1608Metric_Pad1.05x0.95mm_HandSolder
- C17: renamed from C14; footprint Capacitor_SMD:C_0805_2012Metric_Pad1.15x1.40mm_HandSolder -> Capacitor_SMD:C_0603_1608Metric_Pad1.05x0.95mm_HandSolder
- C18: renamed from C15; footprint Capacitor_SMD:C_0805_2012Metric_Pad1.15x1.40mm_HandSolder -> Capacitor_SMD:C_0603_1608Metric_Pad1.05x0.95mm_HandSolder
- C19: renamed from C13; footprint Capacitor_SMD:C_0805_2012Metric_Pad1.15x1.40mm_HandSolder -> Capacitor_SMD:C_0603_1608Metric_Pad1.05x0.95mm_HandSolder
- C2: renamed from C3; value C -> 0.47u; footprint Capacitor_SMD:C_0805_2012Metric_Pad1.15x1.40mm_HandSolder -> Capacitor_SMD:C_0603_1608Metric_Pad1.05x0.95mm_HandSolder
- C4: footprint Capacitor_SMD:C_0805_2012Metric_Pad1.15x1.40mm_HandSolder -> Capacitor_SMD:C_0603_1608Metric_Pad1.05x0.95mm_HandSolder
- C7: renamed from C5; footprint Capacitor_SMD:C_1206_3216Metric_Pad1.42x1.75mm_HandSolder -> Capacitor_SMD:C_0603_1608Metric_Pad1.05x0.95mm_HandSolder
- C8: renamed from C6; footprint Capacitor_SMD:C_0805_2012Metric_Pad1.15x1.40mm_HandSolder -> Capacitor_SMD:C_0603_1608Metric_Pad1.05x0.95mm_HandSolder
- C9: renamed from C7; footprint Capacitor_SMD:C_0805_2012Metric_Pad1.15x1.40mm_HandSolder -> Capacitor_SMD:C_0603_1608Metric_Pad1.05x0.95mm_HandSolder
- J1: value Barrel_Jack_Switch -> Conn_01x02_Male; footprint Connector_PinHeader_2.54mm:PinHeader_1x03_P2.54mm_Vertical -> Connector_PinHeader_2.54mm:PinHeader_1x02_P2.54mm_Vertical
- J3: value AudioJack3 -> Conn_01x02_Female; footprint Connector_PinHeader_2.54mm:PinHeader_1x03_P2.54mm_Vertical -> Connector_PinHeader_2.54mm:PinHeader_1x02_P2.54mm_Vertical; moved to B.Cu
- J4: value Conn_01x02_Male -> AudioJack3_SwitchTR; footprint Connector_PinHeader_2.54mm:PinHeader_1x02_P2.54mm_Vertical -> Connector_PinHeader_2.54mm:PinHeader_1x05_P2.54mm_Vertical; moved to B.Cu
- R10: renamed from R8; footprint Resistor_SMD:R_1206_3216Metric_Pad1.42x1.75mm_HandSolder -> Resistor_SMD:R_0603_1608Metric_Pad1.05x0.95mm_HandSolder
- R13: renamed from R9; footprint Resistor_SMD:R_0805_2012Metric_Pad1.15x1.40mm_HandSolder -> Resistor_SMD:R_0603_1608Metric_Pad1.05x0.95mm_HandSolder
- R14: renamed from R10; footprint Resistor_SMD:R_0805_2012Metric_Pad1.15x1.40mm_HandSolder -> Resistor_SMD:R_0603_1608Metric_Pad1.05x0.95mm_HandSolder
- R15: renamed from R11; footprint Resistor_SMD:R_0805_2012Metric_Pad1.15x1.40mm_HandSolder -> Resistor_SMD:R_0603_1608Metric_Pad1.05x0.95mm_HandSolder
- R16: renamed from R12; footprint Resistor_SMD:R_0805_2012Metric_Pad1.15x1.40mm_HandSolder -> Resistor_SMD:R_0603_1608Metric_Pad1.05x0.95mm_HandSolder
- R17: renamed from R14; footprint Resistor_SMD:R_0805_2012Metric_Pad1.15x1.40mm_HandSolder -> Resistor_SMD:R_0603_1608Metric_Pad1.05x0.95mm_HandSolder
- R18: renamed from R15; footprint Resistor_SMD:R_0805_2012Metric_Pad1.15x1.40mm_HandSolder -> Resistor_SMD:R_0603_1608Metric_Pad1.05x0.95mm_HandSolder
- R19: renamed from R13; footprint Resistor_SMD:R_0805_2012Metric_Pad1.15x1.40mm_HandSolder -> Resistor_SMD:R_0603_1608Metric_Pad1.05x0.95mm_HandSolder
- R2: value R -> 150; footprint Resistor_SMD:R_0805_2012Metric_Pad1.15x1.40mm_HandSolder -> Resistor_SMD:R_0603_1608Metric_Pad1.05x0.95mm_HandSolder
- R20: renamed from R16; footprint Resistor_SMD:R_0805_2012Metric_Pad1.15x1.40mm_HandSolder -> Resistor_SMD:R_0603_1608Metric_Pad1.05x0.95mm_HandSolder
- R21: renamed from R17; footprint Resistor_SMD:R_0805_2012Metric_Pad1.15x1.40mm_HandSolder -> Resistor_SMD:R_0603_1608Metric_Pad1.05x0.95mm_HandSolder
- R22: renamed from R18; footprint Resistor_SMD:R_0805_2012Metric_Pad1.15x1.40mm_HandSolder -> Resistor_SMD:R_0603_1608Metric_Pad1.05x0.95mm_HandSolder
- R23: renamed from R20; footprint Resistor_SMD:R_0805_2012Metric_Pad1.15x1.40mm_HandSolder -> Resistor_SMD:R_0603_1608Metric_Pad1.05x0.95mm_HandSolder
- R24: renamed from R21; footprint Resistor_SMD:R_0805_2012Metric_Pad1.15x1.40mm_HandSolder -> Resistor_SMD:R_0603_1608Metric_Pad1.05x0.95mm_HandSolder
- R25: renamed from R19; footprint Resistor_SMD:R_0805_2012Metric_Pad1.15x1.40mm_HandSolder -> Resistor_SMD:R_0603_1608Metric_Pad1.05x0.95mm_HandSolder
- R4: renamed from R5; footprint Resistor_SMD:R_0805_2012Metric_Pad1.15x1.40mm_HandSolder -> Resistor_SMD:R_0603_1608Metric_Pad1.05x0.95mm_HandSolder
- R5: renamed from R3; footprint Resistor_SMD:R_0805_2012Metric_Pad1.15x1.40mm_HandSolder -> Resistor_SMD:R_0603_1608Metric_Pad1.05x0.95mm_HandSolder
- R6: renamed from R4; footprint Resistor_SMD:R_0805_2012Metric_Pad1.15x1.40mm_HandSolder -> Resistor_SMD:R_0603_1608Metric_Pad1.05x0.95mm_HandSolder
- R7: renamed from R6; value R -> 20k; footprint Resistor_SMD:R_0805_2012Metric_Pad1.15x1.40mm_HandSolder -> Resistor_SMD:R_0603_1608Metric_Pad1.05x0.95mm_HandSolder
- R8: renamed from R7; footprint Resistor_SMD:R_1206_3216Metric_Pad1.42x1.75mm_HandSolder -> Resistor_SMD:R_0603_1608Metric_Pad1.05x0.95mm_HandSolder
- RV2: renamed from RV1; value 10k -> 20k
- Y1: footprint Crystal:Crystal_HC49-U_Vertical -> Crystal:Crystal_SMD_5032-2Pin_5.0x3.2mm_HandSoldering; moved to B.Cu
- moved D5 214.3 mm to (280.8, 25.1), turned to 270 degrees
- moved J3 210.0 mm to (280.8, 69.0)
- moved D1 201.8 mm to (280.8, 35.5), turned to 270 degrees
- moved J4 183.5 mm to (280.8, 62.8)
- moved R3 182.2 mm to (263.1, 20.9), turned to 180 degrees
- moved J1 180.1 mm to (280.8, 49.0), turned to 0 degrees
- moved U3 165.8 mm to (264.9, 26.1), turned to 270 degrees
- moved R10 153.3 mm to (266.9, 31.5), turned to 90 degrees
- moved C7 151.9 mm to (266.0, 21.6)
- moved R8 151.4 mm to (265.4, 31.5), turned to 90 degrees
- moved L1 147.4 mm to (273.2, 27.4), turned to 270 degrees
- moved C12 137.8 mm to (263.9, 37.6), turned to 0 degrees
- moved U2 132.3 mm to (271.4, 67.0), turned to 0 degrees
- moved C4 131.7 mm to (275.9, 67.2), turned to 90 degrees
- moved R7 129.5 mm to (271.4, 63.5), turned to 180 degrees
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- renumbered C9 to C12, D2 to D3, R1 to R3, SW2 to SW1, SW4 to SW2, SW5 to SW3, SW3 to SW4, U3 to U2, U2 to U3
Connections:
- C14 pad 1: Net-(C10-Pad1) (its old number) -> Net-(C14-Pad1)
- C15 pad 1: Net-(C11-Pad1) (its old number) -> Net-(C15-Pad1)
- C16 pad 1: Net-(C12-Pad1) -> Net-(C16-Pad1)
- C17 pad 1: Net-(C14-Pad1) -> Net-(C17-Pad1)
- C18 pad 1: Net-(C15-Pad1) -> Net-(C18-Pad1)
- C19 pad 1: Net-(C13-Pad1) -> Net-(C19-Pad1)
- C4 pad 1: Net-(C4-Pad1) -> GND
- C4 pad 2: GND -> +5V
- D1 pad 1: Net-(D1-Pad1) -> +9V
- J1 pad 1: Net-(J1-Pad1) -> GND
- J2 pad 1: +5V -> GND
- J2 pad 2: NRST -> +5V
- J2 pad 3: GND -> NRST
- J2 pad 4: SPI_SCK -> SPI_MISO
- J2 pad 5: SPI_MISO -> SPI_SCK
- J3 pad 1: (no net) -> Net-(J3-Pad1)
- J3 pad 2: (no net) -> Net-(J3-Pad2)
- R20 pad 2: Net-(C10-Pad1) (its old number) -> Net-(C14-Pad1)
- R21 pad 1: Net-(C11-Pad1) (its old number) -> Net-(C15-Pad1)
- R22 pad 1: Net-(C12-Pad1) -> Net-(C16-Pad1)
- R23 pad 1: Net-(C14-Pad1) -> Net-(C17-Pad1)
- R24 pad 1: Net-(C15-Pad1) -> Net-(C18-Pad1)
- R25 pad 2: Net-(C13-Pad1) -> Net-(C19-Pad1)
- R4 pad 1: Net-(D4-Pad2) -> Net-(R4-Pad1)
- R4 pad 2: Net-(R5-Pad2) -> Net-(D2-Pad2)
- R5 pad 2: Net-(R3-Pad2) -> Net-(R5-Pad2)
- R6 pad 2: Net-(D3-Pad2) (its old number) -> Net-(D4-Pad2)
- SW1 pad MP: (no net) -> GND
- U1 pad 23: DIG3 -> DIG0
- U1 pad 24: DIG2 -> DIG1
- U1 pad 25: DIG1 -> DIG2
- U1 pad 26: DIG0 -> DIG3
- U1 pad 27: AMP_SHUTDOWN -> (no net)
- U1 pad 28: (no net) -> AMP_SHUTDOWN
- U1 pad 30: Net-(R3-Pad2) -> Net-(R4-Pad1)
- U2 pad 2: Net-(C4-Pad1) -> Net-(C6-Pad1)
- U2 pad 3: Net-(C4-Pad1) -> Net-(C6-Pad1)
- U5 pad 1: Net-(C13-Pad1) -> Net-(C17-Pad1)
- U5 pad 11: Net-(C12-Pad1) -> Net-(C14-Pad1)
- U5 pad 12: ENC_A -> ENC_BUTTON
- U5 pad 13: Net-(C10-Pad1) (its old number) -> Net-(C15-Pad1)
- U5 pad 3: Net-(C14-Pad1) -> Net-(C18-Pad1)
- U5 pad 5: Net-(C11-Pad1) (its old number) -> Net-(C19-Pad1)
- U5 pad 6: ENC_BUTTON -> BUTTON2
- U5 pad 8: BUTTON2 -> ENC_A
- U5 pad 9: Net-(C15-Pad1) -> Net-(C16-Pad1)
Routing:
- net +5V: track 152.9 -> 230.0 mm
- net GND: track 19.1 -> 81.9 mm, vias 2 -> 10
- net +9V: track 0.00 -> 42.2 mm, vias 0 -> 2
- net Net-(R3-Pad2): track 40.7 -> 0.00 mm
- net Net-(C17-Pad1): track 0.00 -> 40.4 mm, vias 0 -> 5
- net BUTTON2: track 41.3 -> 4.80 mm
- net Net-(C13-Pad1): track 35.7 -> 0.00 mm, vias 2 -> 0
- net Net-(R4-Pad1): track 0.00 -> 33.8 mm, vias 0 -> 2
- net Net-(C12-Pad1): track 28.7 -> 0.00 mm
- net Net-(C18-Pad1): track 0.00 -> 28.0 mm
- net SOUND_OUT: track 33.0 -> 58.8 mm
- net DIG0: track 33.0 -> 9.70 mm
- net NRST: track 44.3 -> 22.3 mm, vias 1 -> 2
- net BUTTON1: track 26.5 -> 5.24 mm
- net (no net): track 21.0 -> 0.00 mm, vias 4 -> 0
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- removed copper zone on F.Cu, net GND
Other:
- board size 127.2 x 85.4 mm -> 60 x 66.6 mm
- net class Default: trace_width 0.5 -> 0.25; via_dia 1.1 -> 0.4; via_drill 0.5 -> 0.3
- net class Power added: clearance 0.2, trace_width 0.5, via_dia 1, via_drill 0.6
- net class Sound added: clearance 0.2, trace_width 0.5, via_dia 1, via_drill 0.6
- board text added: "+5V"
- board text added: "+9V"
- board text added: "GND"
- board text added: "JLCJLCJLCJLC"
- board text added: "MISO"
- board text added: "NRST"
- board text added: "R"
- board text added: "RN"
- board text added: "S"
- board text added: "SCK"
- board text added: "SPKR"
- board text added: "T"
- board text added: "TN"
- board text added: "mtrnm 2.1"

Commit message: Change pot polarity
Parts:
- turned R11 to 270 degrees
- turned R12 to 90 degrees
Connections:
- RV1 pad 1: Net-(C10-Pad2) -> GND
- RV1 pad 3: GND -> Net-(C10-Pad2)
- RV1 pad 4: Net-(C11-Pad2) -> GND
- RV1 pad 6: GND -> Net-(C11-Pad2)
Routing:
- net GND: track 81.9 -> 71.4 mm, vias 10 -> 9
- net Net-(C10-Pad2): track 9.64 -> 16.3 mm
- net Net-(J4-PadT): track 12.6 -> 13.9 mm
- net Net-(C11-Pad2): track 7.40 -> 6.44 mm
- net Net-(C10-Pad1): track 23.7 -> 23.0 mm
Other:
- board text added: "mtrnm 2.2"
- board text removed: "mtrnm 2.1"
