File: circuit/schematic.sch (KiCad schematic (older format))
At the start: 62 parts, among them J1 Barrel_Jack_Switch, J2 Conn_01x05_Male, J3 AudioJack3, J4 Conn_01x02_Male, SW1 SW_DPDT_x2, SW2 Rotary_Encoder_Switch, SW3 SW_Push, SW4 SW_Push, SW5 SW_Push, U1 ATmega328-AU, U2 MC33063AD, U3 SSM2211S, U4 STP08CP05, U5 74HC14, U6 CC56-12SRWA, Y1 16M

Commit message: Update board
Parts:
- removed BT1: 9V, Connector_PinHeader_2.54mm:PinHeader_1x02_P2.54mm_Vertical, symbol Device:Battery
- removed J1: Barrel_Jack_Switch, Connector_PinHeader_2.54mm:PinHeader_1x03_P2.54mm_Vertical, symbol Connector:Barrel_Jack_Switch
- removed J3: AudioJack3, Connector_PinHeader_2.54mm:PinHeader_1x03_P2.54mm_Vertical, symbol Connector:AudioJack3
- removed J4: Conn_01x02_Male, Connector_PinHeader_2.54mm:PinHeader_1x02_P2.54mm_Vertical, symbol Connector:Conn_01x02_Male
- removed LS1: Speaker, Connector_PinHeader_2.54mm:PinHeader_1x02_P2.54mm_Vertical, symbol Device:Speaker
- removed SW1: SW_DPDT_x2, Button_Switch_THT:SMTS-202-A2, symbol Switch:SW_DPDT_x2
- added C10, C3: 220u, Capacitor_THT:CP_Radial_D8.0mm_P3.50mm, symbol Device:CP
- added C13, C4: 0.1u, Capacitor_SMD:C_0603_1608Metric_Pad1.05x0.95mm_HandSolder, symbol Device:C
- added H1, H2, H3, H4: MountingHole, MountingHole:MountingHole_3.2mm_M3, symbol Mechanical:MountingHole
- added J1: Conn_01x02_Male, Connector_PinHeader_2.54mm:PinHeader_1x02_P2.54mm_Vertical, symbol Connector:Conn_01x02_Male
- added J3: Conn_01x02_Female, Connector_PinHeader_2.54mm:PinHeader_1x02_P2.54mm_Vertical, symbol Connector:Conn_01x02_Female
- added J4: AudioJack3_SwitchTR, Connector_PinHeader_2.54mm:PinHeader_1x05_P2.54mm_Vertical, symbol Connector:AudioJack3_SwitchTR
- added R1: 5k, Resistor_SMD:R_0603_1608Metric_Pad1.05x0.95mm_HandSolder, symbol Device:R
- added R11, R12: 4.7k, Resistor_SMD:R_0603_1608Metric_Pad1.05x0.95mm_HandSolder, symbol Device:R
- added RV1: R_POT_Dual, Potentiometer_THT:Potentiometer_Alps_RK09L_Double_Vertical, symbol Device:R_POT_Dual
- C1: footprint Capacitor_SMD:C_0805_2012Metric_Pad1.15x1.40mm_HandSolder -> Capacitor_SMD:C_0603_1608Metric
- C14: renamed from C10; footprint Capacitor_SMD:C_0805_2012Metric_Pad1.15x1.40mm_HandSolder -> Capacitor_SMD:C_0603_1608Metric_Pad1.05x0.95mm_HandSolder
- C15: renamed from C11; footprint Capacitor_SMD:C_0805_2012Metric_Pad1.15x1.40mm_HandSolder -> Capacitor_SMD:C_0603_1608Metric_Pad1.05x0.95mm_HandSolder
- C16: renamed from C12; footprint Capacitor_SMD:C_0805_2012Metric_Pad1.15x1.40mm_HandSolder -> Capacitor_SMD:C_0603_1608Metric_Pad1.05x0.95mm_HandSolder
- C17: renamed from C14; footprint Capacitor_SMD:C_0805_2012Metric_Pad1.15x1.40mm_HandSolder -> Capacitor_SMD:C_0603_1608Metric_Pad1.05x0.95mm_HandSolder
- C18: renamed from C15; footprint Capacitor_SMD:C_0805_2012Metric_Pad1.15x1.40mm_HandSolder -> Capacitor_SMD:C_0603_1608Metric_Pad1.05x0.95mm_HandSolder
- C19: renamed from C13; footprint Capacitor_SMD:C_0805_2012Metric_Pad1.15x1.40mm_HandSolder -> Capacitor_SMD:C_0603_1608Metric_Pad1.05x0.95mm_HandSolder
- C2: renamed from C3; value C -> 0.47u; footprint Capacitor_SMD:C_0805_2012Metric_Pad1.15x1.40mm_HandSolder -> Capacitor_SMD:C_0603_1608Metric_Pad1.05x0.95mm_HandSolder
- C6: renamed from C4; footprint Capacitor_SMD:C_0805_2012Metric_Pad1.15x1.40mm_HandSolder -> Capacitor_SMD:C_0603_1608Metric_Pad1.05x0.95mm_HandSolder
- C7: renamed from C5; footprint Capacitor_SMD:C_1206_3216Metric_Pad1.42x1.75mm_HandSolder -> Capacitor_SMD:C_0603_1608Metric_Pad1.05x0.95mm_HandSolder
- C8: renamed from C6; footprint Capacitor_SMD:C_0805_2012Metric_Pad1.15x1.40mm_HandSolder -> Capacitor_SMD:C_0603_1608Metric_Pad1.05x0.95mm_HandSolder
- C9: renamed from C7; footprint Capacitor_SMD:C_0805_2012Metric_Pad1.15x1.40mm_HandSolder -> Capacitor_SMD:C_0603_1608Metric_Pad1.05x0.95mm_HandSolder
- R10: renamed from R8; footprint Resistor_SMD:R_1206_3216Metric_Pad1.42x1.75mm_HandSolder -> Resistor_SMD:R_0603_1608Metric_Pad1.05x0.95mm_HandSolder
- R13: renamed from R9; footprint Resistor_SMD:R_0805_2012Metric_Pad1.15x1.40mm_HandSolder -> Resistor_SMD:R_0603_1608Metric_Pad1.05x0.95mm_HandSolder
- R14: renamed from R10; footprint Resistor_SMD:R_0805_2012Metric_Pad1.15x1.40mm_HandSolder -> Resistor_SMD:R_0603_1608Metric_Pad1.05x0.95mm_HandSolder
- R15: renamed from R11; footprint Resistor_SMD:R_0805_2012Metric_Pad1.15x1.40mm_HandSolder -> Resistor_SMD:R_0603_1608Metric_Pad1.05x0.95mm_HandSolder
- R16: renamed from R12; footprint Resistor_SMD:R_0805_2012Metric_Pad1.15x1.40mm_HandSolder -> Resistor_SMD:R_0603_1608Metric_Pad1.05x0.95mm_HandSolder
- R17: renamed from R14; footprint Resistor_SMD:R_0805_2012Metric_Pad1.15x1.40mm_HandSolder -> Resistor_SMD:R_0603_1608Metric_Pad1.05x0.95mm_HandSolder
- R18: renamed from R15; footprint Resistor_SMD:R_0805_2012Metric_Pad1.15x1.40mm_HandSolder -> Resistor_SMD:R_0603_1608Metric_Pad1.05x0.95mm_HandSolder
- R19: renamed from R13; footprint Resistor_SMD:R_0805_2012Metric_Pad1.15x1.40mm_HandSolder -> Resistor_SMD:R_0603_1608Metric_Pad1.05x0.95mm_HandSolder
- R2: value R -> 150; footprint Resistor_SMD:R_0805_2012Metric_Pad1.15x1.40mm_HandSolder -> Resistor_SMD:R_0603_1608Metric_Pad1.05x0.95mm_HandSolder
- R20: renamed from R16; footprint Resistor_SMD:R_0805_2012Metric_Pad1.15x1.40mm_HandSolder -> Resistor_SMD:R_0603_1608Metric_Pad1.05x0.95mm_HandSolder
- R21: renamed from R17; footprint Resistor_SMD:R_0805_2012Metric_Pad1.15x1.40mm_HandSolder -> Resistor_SMD:R_0603_1608Metric_Pad1.05x0.95mm_HandSolder
- R22: renamed from R18; footprint Resistor_SMD:R_0805_2012Metric_Pad1.15x1.40mm_HandSolder -> Resistor_SMD:R_0603_1608Metric_Pad1.05x0.95mm_HandSolder
- R23: renamed from R20; footprint Resistor_SMD:R_0805_2012Metric_Pad1.15x1.40mm_HandSolder -> Resistor_SMD:R_0603_1608Metric_Pad1.05x0.95mm_HandSolder
- R24: renamed from R21; footprint Resistor_SMD:R_0805_2012Metric_Pad1.15x1.40mm_HandSolder -> Resistor_SMD:R_0603_1608Metric_Pad1.05x0.95mm_HandSolder
- R25: renamed from R19; footprint Resistor_SMD:R_0805_2012Metric_Pad1.15x1.40mm_HandSolder -> Resistor_SMD:R_0603_1608Metric_Pad1.05x0.95mm_HandSolder
- R4: renamed from R5; footprint Resistor_SMD:R_0805_2012Metric_Pad1.15x1.40mm_HandSolder -> Resistor_SMD:R_0603_1608Metric_Pad1.05x0.95mm_HandSolder
- R5: renamed from R3; footprint Resistor_SMD:R_0805_2012Metric_Pad1.15x1.40mm_HandSolder -> Resistor_SMD:R_0603_1608Metric_Pad1.05x0.95mm_HandSolder
- R6: renamed from R4; footprint Resistor_SMD:R_0805_2012Metric_Pad1.15x1.40mm_HandSolder -> Resistor_SMD:R_0603_1608Metric_Pad1.05x0.95mm_HandSolder
- R7: renamed from R6; value R -> 20k; footprint Resistor_SMD:R_0805_2012Metric_Pad1.15x1.40mm_HandSolder -> Resistor_SMD:R_0603_1608Metric_Pad1.05x0.95mm_HandSolder
- R8: renamed from R7; footprint Resistor_SMD:R_1206_3216Metric_Pad1.42x1.75mm_HandSolder -> Resistor_SMD:R_0603_1608Metric_Pad1.05x0.95mm_HandSolder
- R9: renamed from R22; footprint Resistor_SMD:R_0805_2012Metric_Pad1.15x1.40mm_HandSolder -> Resistor_SMD:R_0603_1608Metric_Pad1.05x0.95mm_HandSolder
- RV2: renamed from RV1; value 10k -> 20k
- Y1: footprint Crystal:Crystal_HC49-U_Vertical -> Crystal:Crystal_SMD_5032-2Pin_5.0x3.2mm_HandSoldering
- renumbered C8 to C11, C9 to C12, C2 to C5, D4 to D2, D2 to D3, D3 to D4, R1 to R3, SW2 to SW1, SW4 to SW2, SW5 to SW3, SW3 to SW4, U3 to U2, U2 to U3
Connections:
- wire segments 169 -> 219
- no-connect marks 6 -> 5
Other:
- note added: "27\n1.2\n"
- note added: "MIDI OUT?\n"
- note added: "Speaker"
- note removed: "hdphn detect?\n"
- moved on the sheet: C17, C18, C19, C2, C7, D1, D2, D3, R10, R17, R18, R19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

Commit message: Change pot polarity
Connections:
- wire segments 219 -> 216
Other:
- note added: "3\n1"
- note added: "6\n4\n"
Changed lines of the file:
@@
 L Device:CP C11
 U 1 1 5EC94855
-P 4200 5600
-F 0 "C11" V 4455 5600 50  0000 C CNN
-F 1 "220u" V 4364 5600 50  0000 C CNN
-F 2 "Capacitor_THT:CP_Radial_D8.0mm_P3.50mm" H 4238 5450 50  0001 C CNN
-F 3 "~" H 4200 5600 50  0001 C CNN
-	1    4200 5600
+P 4200 5950
+F 0 "C11" V 4455 5950 50  0000 C CNN
+F 1 "220u" V 4364 5950 50  0000 C CNN
+F 2 "Capacitor_THT:CP_Radial_D8.0mm_P3.50mm" H 4238 5800 50  0001 C CNN
+F 3 "~" H 4200 5950 50  0001 C CNN
+	1    4200 5950
 	0    -1   -1   0
 $EndComp
@@
 L Device:CP C10
 U 1 1 600F1B99
-P 4200 5100
-F 0 "C10" V 4455 5100 50  0000 C CNN
-F 1 "220u" V 4364 5100 50  0000 C CNN
-F 2 "Capacitor_THT:CP_Radial_D8.0mm_P3.50mm" H 4238 4950 50  0001 C CNN
-F 3 "~" H 4200 5100 50  0001 C CNN
-	1    4200 5100
+P 4200 5450
+F 0 "C10" V 4455 5450 50  0000 C CNN
+F 1 "220u" V 4364 5450 50  0000 C CNN
+F 2 "Capacitor_THT:CP_Radial_D8.0mm_P3.50mm" H 4238 5300 50  0001 C CNN
+F 3 "~" H 4200 5450 50  0001 C CNN
+	1    4200 5450
 	0    -1   -1   0
 $EndComp
@@
 	2950 5100 2950 5650
 Wire Wire Line
-	4350 5100 4800 5100
-Wire Wire Line
-	4800 5100 4800 5150
-Wire Wire Line
-	3800 5950 3950 5950
-Wire Wire Line
-	4800 5650 4800 5600
-Wire Wire Line
-	4800 5600 4350 5600
-Wire Wire Line
-	3950 5600 4050 5600
-Wire Wire Line
-	3950 5600 3950 5950
-Wire Wire Line
-	3850 5750 3850 5100
-Connection ~ 3850 5100
-Wire Wire Line
-	3850 5100 4050 5100
-Wire Wire Line
-	4800 5450 4800 5550
-Wire Wire Line
-	4800 5550 4700 5550
-Wire Wire Line
-	4700 5550 4700 6050
-Wire Wire Line
-	4700 6050 4800 6050
-Wire Wire Line
-	4800 6050 4800 5950
-Wire Wire Line
-	4700 6050 4700 6400
-Wire Wire Line
-	4700 6400 3300 6400
-Connection ~ 4700 6050
+	3850 5750 3850 5450
 Connection ~ 3300 6400
 Wire Wire Line
@@
 Wire Wire Line
 	5100 6150 5100 6400
-Connection ~ 4700 6400
 Wire Wire Line
 	5100 5650 5100 5700
@@
 Wire Wire Line
 	5200 5700 5200 6400
-Wire Wire Line
-	4700 6400 5100 6400
 Connection ~ 5100 6400
 Wire Wire Line
@@
 Wire Wire Line
 	6650 2500 6850 2500
+Text Notes 4850 5100 0    50   ~ 0
+3\n1
+Text Notes 4550 5900 0    50   ~ 0
+6\n4\n
+Wire Wire Line
+	3300 6400 4600 6400
+Wire Wire Line
+	4800 5450 4350 5450
+Wire Wire Line
+	4350 5950 4800 5950
+Wire Wire Line
+	4800 5650 4800 5600
+Wire Wire Line
+	4800 5600 4600 5600
+Wire Wire Line
+	4600 5600 4600 6400
+Connection ~ 4600 6400
+Wire Wire Line
+	4600 6400 5100 6400
+Wire Wire Line
+	4800 5150 4800 5100
+Wire Wire Line
+	4800 5100 4600 5100
+Wire Wire Line
+	4600 5100 4600 5600
+Connection ~ 4600 5600
+Wire Wire Line
+	4050 5450 3850 5450
+Connection ~ 3850 5450
+Wire Wire Line
+	3850 5450 3850 5100
+Wire Wire Line
+	3800 5950 4050 5950
 $EndSCHEMATC
